File: EAGLE/projects/HMD/ESP32.sch (EAGLE design)
At the start: 10 parts, among them J1 CORTEX_DEBUG_PTH

Commit message: PCB layed out
Parts:
- removed R2, R3, R4: (no value), SparkFun-Resistors:RESISTOR0603
- added C10, C11, C13: 4.7uF, SparkFun-Capacitors:4.7UF0603
- added C12, C9: 2.2uF, SparkFun-Capacitors:2.2UF-0603-10V-20%
- added C14, C8: 10µF, microbuilder:CAP_CERAMIC_0603
- added C7: 0.1uF, microbuilder:CAP_CERAMIC_0603MP
- added D1: RED, SparkFun-LED:LED-RED0603
- added D2: 1N4004, diode:1N4004
- added D3: 1N4148, microbuilder:DIODESOD-323
- added J2: (no value), SparkFun-Connectors:CONN_08"
- added J3: (no value), SparkFun-Connectors:CONN_05
- added Q3, Q4: BSS138, microbuilder:MOSFET-NWIDE
- added R10: 10k, SparkFun-Resistors:RESISTOR0603
- added R11, R12: 100k, SparkFun-Resistors:RESISTOR0603
- added R13: 3.3M, SparkFun-Resistors:RESISTOR0603
- added R14, R15, R16, R17, R18, R19: 10K, microbuilder:RESISTOR_0603
- added R8: 470, SparkFun-Resistors:RESISTOR0603
- added R9: 12k, SparkFun-Resistors:RESISTOR0603
- added S1: MOMENTARY-SWITCH-SPST-PTH-6.0MM, SparkFun-Switches:MOMENTARY-SWITCH-SPST-PTH-6.0MM
- added U$5: MCP6001-X_SOT-23-5, HMD_Library:MCP6001-X_SOT-23-5
- added U$6: ADPS_9008_020, HMD_Library:ADPS_9008_020
- added U$7: KB_REVMNT_LED, HMD_Library:KB_REVMNT_LED
- added U3: LIS3DHTR, microbuilder:ACCEL_LIS3DHTR
- added U4: MIC5225-3.3, microbuilder:VREG_SOT23-5
- J1: value CORTEX_DEBUG_PTH -> (none); device SparkFun-Connectors:CORTEX_DEBUG_PTH -> SparkFun-Connectors:CONN_04
- R1: value (none) -> 470
- R5: value (none) -> 10k
Connections:
- removed net MTCK: R2.2, U$1.IO13
- removed net MTDI: R4.2, U$1.IO12
- removed net MTDO: R3.2, U$1.IO15
- removed net MTMS: R1.2, U$1.IO14
- removed net N$3: J1.NC/TDI, R4.1
- removed net N$4: J1.SWO/TDO, R3.1
- new net BUSY: J2.8, U$1.IO22
- new net CS: J2.5, U$1.IO19
- new net CS_IMU: D3.C
- new net DC: J2.6, U$1.IO21
- new net DIN: J2.3, U$1.IO5
- new net HR_OUT: R13.2, U$1.SENSOR_VP, U$5.VOUT
- new net INT1: U3.INT1
- new net N$10: C10.2, C11.1, C13.2
- new net N$11: C11.2, C12.1, R10.2
- new net N$14: C12.2, R11.2, R12.1, U$5.VIN+
- new net N$15: R10.1, R13.1, U$5.VIN-
- new net N$16: D2.C, U$5.VDD, U$6.VCC
- new net N$17: R8.2, U$7.C
- new net N$7: J1.1, U$1.IO0
- new net N$9: C10.1, R9.2, U$6.OUT
- new net PRX: J1.3, U$1.TXD0
- new net PTX: J1.2, U$1.RXD0
- new net RST: J2.7, U$1.IO23
- new net SCL: J3.4, Q4.D, R18.1, U$1.IO17
- new net SCL_3.3V: Q4.S, R16.1, U3.SCL
- new net SDA: J3.5, Q3.D, R17.1, U$1.IO16
- new net SDA_3.3V: Q3.S, R15.1, U3.SDA
- new net SDO: R19.2, U3.SDO
- new net SPICLK: J2.4, U$1.IO18
- new net VIN: C14.1, J3.1, R17.2, R18.2, U4.EN, U4.IN
- net 3.3V: now also C7.1, C8.1, C9.1, D1.A, D2.A, J2.1, J3.2, Q3.G, Q4.G, R11.1, R14.2, R15.2, R16.2, U$7.A, U3.VDD, U3.VDDIO, U4.OUT
- net EN: now also J1.4, S1.2
- net GND: now also C13.1, C14.2, C7.2, C8.2, C9.2, J2.2, J3.3, R1.1, R12.2, R19.1, R8.1, R9.1, S1.1, U$5.VSS, U$6.GND, U3.GND@1, U3.GND@2, U3.RES(GND), U4.GND
- net N$1: now also D3.A, R14.1, U3.CS; no longer J1.SWDIO/TMS, R1.1
- net N$2: now also D1.C, R1.2; no longer J1.SWDCLK/TCK, R2.1
Other:
- moved on the sheet: C1, C2, C3, R1, R5, U$1
