File: EAGLE/projects/HMD/ESP32.sch (EAGLE design)
At the start: 40 parts, among them Q3 BSS138, Q4 BSS138, U3 LIS3DHTR, U4 MIC5225-3.3

Commit message: Revert "Version 1 micro"
This reverts commit 22c8d65d876e5e97d8f3c243cdc0f8aa191d734f.
Parts:
- removed U$8: DI0603, HMD_Library:DI0603
- added D2: 1N4004, diode:1N4004
Connections:
- removed net HR_IN: C9.1, R11.1, U$1.IO13, U$7.A, U$8.P$2
- net 3.3V: now also C9.1, D2.A, R11.1, U$7.A
- net N$16: now also D2.C; no longer U$8.P$1
Other:
- note removed: "ACCELEROMETER"
- note removed: "ESP WROOM 32 SCHEMATIC"
- note removed: "I2C HEADERS"
- note removed: "LIGHT SENSOR"
- note removed: "OPERATIONAL AMPLIFIER"
- note removed: "PROGRAMMING HEADERS"
- note removed: "PULSE HEARTEATE SENSOR"
- note removed: "RESET CIRCUITRY"
- note removed: "SIGNAL REGULATOR"
- note removed: "SPI HEADERS"
- note removed: "TEST LED"
- note removed: "VOLTAGE REGULATOR"
- moved on the sheet: C1, C10, C11, C12, C13, C14, C2, C3, C7, C8, C9, D1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

Commit message: Version 1 micro
Parts:
- removed D2: 1N4004, diode:1N4004
- added U$8: DI0603, HMD_Library:DI0603
Connections:
- new net HR_IN: C9.1, R11.1, U$1.IO13, U$7.A, U$8.P$2
- net 3.3V: no longer C9.1, D2.A, R11.1, U$7.A
- net N$16: now also U$8.P$1; no longer D2.C
Other:
- note added: "ACCELEROMETER"
- note added: "ESP WROOM 32 SCHEMATIC"
- note added: "I2C HEADERS"
- note added: "LIGHT SENSOR"
- note added: "OPERATIONAL AMPLIFIER"
- note added: "PROGRAMMING HEADERS"
- note added: "PULSE HEARTEATE SENSOR"
- note added: "RESET CIRCUITRY"
- note added: "SIGNAL REGULATOR"
- note added: "SPI HEADERS"
- note added: "TEST LED"
- note added: "VOLTAGE REGULATOR"
- moved on the sheet: C1, C10, C11, C12, C13, C14, C2, C3, C7, C8, C9, D1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
