File: EAGLE/projects/HMD/coin20mm_updated.brd (EAGLE design)
At the start: 43 x 38.5 mm, 6 parts, among them CN1 1X4-CLEANBIG

Commit message: working LIS3dh code, cloud updates
Parts:
- removed FID1, FID2: FIDUCIAL"", microbuilder:FIDUCIAL_1MM
- removed U$6: (no value), microbuilder:SYMBOL_PLUS
- removed U$7: (no value), microbuilder:SYMBOL_MINUS
Routing:
- removed copper zone on layer 1, net GND
Changed lines of the file:
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@@
 </autorouter>
 <elements>
-<element name="FID1" library="microbuilder" package="FIDUCIAL_1MM" value="FIDUCIAL&quot;&quot;" x="5.334" y="5.334" smashed="yes" rot="R270">
-<attribute name="BOM" value="EXCLUDE" x="5.334" y="5.334" size="1.778" layer="27" rot="R270" display="off"/>
-</element>
-<element name="FID2" library="microbuilder" package="FIDUCIAL_1MM" value="FIDUCIAL&quot;&quot;" x="40.002" y="29.128" smashed="yes" rot="R270">
-<attribute name="BOM" value="EXCLUDE" x="40.002" y="29.128" size="1.778" layer="27" rot="R270" display="off"/>
-</element>
 <element name="B1" library="microbuilder" package="CR2032_SMT_BAT-HLD-001" value="" x="32.255" y="20.492" smashed="yes" rot="R90">
-<attribute name="VALUE" x="40.615" y="10.078" size="0.4064" layer="27" font="vector" ratio="10" rot="R90"/>
+<attribute name="VALUE" x="40.615" y="10.078" size="0.4064" layer="16" font="vector" ratio="10" rot="R90"/>
 </element>
 <element name="CN1" library="adafruit2" package="1X04-CLEANBIG" value="1X4-CLEANBIG" x="2.9" y="17.65" smashed="yes" rot="R90"/>
-<element name="U$6" library="microbuilder" package="SYMBOL_PLUS" value="" x="2.878" y="24.315" smashed="yes" rot="R270"/>
-<element name="U$7" library="microbuilder" package="SYMBOL_MINUS" value="" x="2.778" y="11.077" smashed="yes" rot="R270"/>
 </elements>
 <signals>
@@
 <wire x1="24.363" y1="12.6" x2="4.14" y2="12.6" width="1.016" layer="1"/>
 <wire x1="2.9" y1="13.84" x2="4.14" y2="12.6" width="1.016" layer="1"/>
-<polygon width="0" layer="1" isolate="0.4064">
-<vertex x="0.8" y="35.1"/>
-<vertex x="42.7" y="35.1"/>
-<vertex x="42.7" y="35"/>
-<vertex x="42.7" y="6.9"/>
-<vertex x="1" y="6.9"/>
-<vertex x="0.8" y="6.9"/>
-</polygon>
 </signal>
 <signal name="VCC">
