File: EAGLE/projects/HMD/coin20mm_updated.sch (EAGLE design)
At the start: 4 parts, among them CN1 1X4-CLEANBIG

Commit message: working LIS3dh code, cloud updates
Parts:
- removed FID1, FID2: FIDUCIAL"", microbuilder:FIDUCIAL""
Changed lines of the file:
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@@
 </classes>
 <parts>
-<part name="FID1" library="microbuilder" deviceset="FIDUCIAL" device="&quot;&quot;"/>
-<part name="FID2" library="microbuilder" deviceset="FIDUCIAL" device="&quot;&quot;"/>
 <part name="B1" library="microbuilder" deviceset="BATTERY" device="CR2032_BAT-HLD-001"/>
 <part name="CN1" library="adafruit2" deviceset="1X4" device="-CLEANBIG"/>
@@
 </plain>
 <instances>
-<instance part="FID1" gate="G$1" x="243.84" y="48.26" smashed="yes"/>
-<instance part="FID2" gate="G$1" x="251.46" y="48.26" smashed="yes"/>
 <instance part="B1" gate="G$1" x="132.08" y="99.06" smashed="yes" rot="R90">
 <attribute name="NAME" x="128.905" y="99.06" size="1.27" layer="95" rot="R90"/>
